Commit message: Add multiple links script

File: fourLinks.urdf (robot description, URDF)
Before this commit: robot twoLinks, 5 links, 4 joints
Joints:
- joint joint_2_3: axis 1 0 0 -> 0 1 0; child link2 -> link3; origin xyz=0 1 0 rpy=0 -0 0 -> xyz=0 0 1 rpy=0 -0 0; parent link1 -> link2
- joint joint_3_4: axis 1 0 0 -> 0 0 1; child link2 -> link4; origin xyz=0 1 0 rpy=0 -0 0 -> xyz=1 0 0 rpy=0 -0 0; parent link1 -> link3
