Commit message: progress

File: twoLinks.urdf (robot description, URDF)
Before this commit: robot threeLinks, 4 links, 3 joints
Links:
- removed link link3
Joints:
- removed joint joint_2_3
- joint joint_1_2: origin xyz=1 0 0 rpy=0 -0 0 -> xyz=0 0 0 rpy=0 -0 0

Commit message: LL minization finally working

File: twoLinks.urdf (robot description, URDF)
Before this commit: robot twoLinks, 3 links, 2 joints
Links:
- link link1: mass 1 -> 10
- link link2: mass 1 -> 10

Commit message: Results

File: twoLinks.urdf (robot description, URDF)
Before this commit: robot twoLinks, 3 links, 2 joints
Joints:
- joint joint_1_2: axis 1 0 0 -> 0 0 1

Commit message: latest dev

File: twoLinks.urdf (robot description, URDF)
Before this commit: robot twoLinks, 5 links, 4 joints
Links:
- removed link link3
- removed link link4
Joints:
- removed joint joint_2_3
- removed joint joint_3_4
